Commit message: fix gazebo related link names

File: cable_joint_description/urdf/cable_joint.gazebo.xacro (robot description, xacro)
@@ -43,18 +43,18 @@
   <gazebo>
     <plugin filename="libgazebo_ros_force.so" name="gazebo_ros_force">
-      <bodyName>link_cube_northeast</bodyName>
-      <topicName>/force_northeast</topicName>
+      <bodyName>link_northeastCube</bodyName>
+      <topicName>/force_ne</topicName>
     </plugin>
     <plugin filename="libgazebo_ros_force.so" name="gazebo_ros_force">
-      <bodyName>link_cube_northwest</bodyName>
-      <topicName>/force_northwest</topicName>
+      <bodyName>link_northwestCube</bodyName>
+      <topicName>/force_nw</topicName>
     </plugin>
     <plugin filename="libgazebo_ros_force.so" name="gazebo_ros_force">
-      <bodyName>link_cube_southeast</bodyName>
-      <topicName>/force_southeast</topicName>
+      <bodyName>link_southeastCube</bodyName>
+      <topicName>/force_se</topicName>
     </plugin>
     <plugin filename="libgazebo_ros_force.so" name="gazebo_ros_force">
-      <bodyName>link_cube_southwest</bodyName>
-      <topicName>/force_southwest</topicName>
+      <bodyName>link_southwestCube</bodyName>
+      <topicName>/force_sw</topicName>
     </plugin>
   </gazebo>
@@ -62,5 +62,5 @@
     <material>Gazebo/Black</material>
   </gazebo>
-  <gazebo reference="link_camera_body">
+  <gazebo reference="link_cameraBody">
     <material>Gazebo/Red</material>
   </gazebo>
@@ -68,23 +68,23 @@
     <material>Gazebo/Black</material>
   </gazebo>
-  <gazebo reference="link_lower_support">
+  <gazebo reference="link_lowerSupport">
     <material>Gazebo/DarkGrey</material>
   </gazebo>
-  <gazebo reference="link_pin_west">
+  <gazebo reference="link_westPin">
     <material>Gazebo/Yellow</material>
   </gazebo>
-  <gazebo reference="link_pin_east">
+  <gazebo reference="link_eastPin">
     <material>Gazebo/Blue</material>
   </gazebo>
-  <gazebo reference="link_ball_roll">
+  <gazebo reference="link_hiddenLinkRoll">
     <material>Gazebo/White</material>
   </gazebo>
-  <gazebo reference="link_ball_pitch">
+  <gazebo reference="link_hiddenLinkPitch">
     <material>Gazebo/White</material>
   </gazebo>
-  <gazebo reference="link_ball_yaw">
+  <gazebo reference="link_ball">
     <material>Gazebo/Grey</material>
   </gazebo>
-  <gazebo reference="link_upper_support">
+  <gazebo reference="link_upperSupport">
     <material>Gazebo/DarkGrey</material>
   </gazebo>
@@ -92,14 +92,14 @@
     <material>Gazebo/Grey</material>
   </gazebo>
-  <gazebo reference="link_cube_northeast">
+  <gazebo reference="link_northeastCube">
     <material>Gazebo/Turquoise</material>
   </gazebo>
-  <gazebo reference="link_cube_northwest">
+  <gazebo reference="link_northwestCube">
     <material>Gazebo/Gold</material>
   </gazebo>
-  <gazebo reference="link_cube_southwest">
+  <gazebo reference="link_southwestCube">
     <material>Gazebo/Orange</material>
   </gazebo>
-  <gazebo reference="link_cube_southeast">
+  <gazebo reference="link_southeastCube">
     <material>Gazebo/Indigo</material>
   </gazebo>

File: cable_joint_description/urdf/cable_joint.urdf.xacro (robot description, xacro)
@@ -37,5 +37,5 @@
     <xacro:property name="L_DISC" value="0.02"/>
     <xacro:property name="M_DISC" value="0.1"/>
-    <!-- properties of link_camera_body -->
+    <!-- properties of link_cube's -->
     <xacro:property name="L_CUBE" value="0.02"/>
     <xacro:property name="M_CUBE" value="0.001"/>
@@ -73,9 +73,9 @@
         <origin rpy="0 0 ${PI/2}" xyz="0 -0.5 ${L_CAMBODY/2}"/>
         <parent link="world"/>
-        <child link="link_camera_body"/>
+        <child link="link_cameraBody"/>
         <limit effort="0" lower="0" upper="0" velocity="0"/>
         <axis rpy="0 0 0" xyz="0 0 1"/>
     </joint>
-    <link name="link_camera_body">
+    <link name="link_cameraBody">
         <visual>
             <origin rpy="0 0 0" xyz="0 0 0"/>
@@ -99,5 +99,5 @@
     <joint name="joint_camerabody_lens" type="revolute">
         <origin rpy="0 ${PI/2} 0" xyz="${L_CAMBODY/2+L_LENS/2} 0 0"/>
-        <parent link="link_camera_body"/>
+        <parent link="link_cameraBody"/>
         <child link="link_lens"/>
         <limit effort="0" lower="0" upper="0" velocity="0"/>

Commit message: set the existing camera to be the south camera

File: cable_joint_description/urdf/cable_joint.gazebo.xacro (robot description, xacro)
@@ -2,5 +2,5 @@
 <robot>
   <!-- camera -->
-  <gazebo reference="link_optical">
+  <gazebo reference="link_southOptical">
     <sensor type="camera" name="camera1">
       <update_rate>30.0</update_rate>
@@ -31,5 +31,5 @@
         <imageTopicName>image_raw</imageTopicName>
         <cameraInfoTopicName>camera_info</cameraInfoTopicName>
-        <frameName>link_optical</frameName>
+        <frameName>link_southOptical</frameName>
         <hackBaseline>0.07</hackBaseline>
         <distortionK1>0.0</distortionK1>
@@ -59,8 +59,8 @@
     </plugin>
   </gazebo>
-  <gazebo reference="link_lens">
+  <gazebo reference="link_southLens">
     <material>Gazebo/Black</material>
   </gazebo>
-  <gazebo reference="link_cameraBody">
+  <gazebo reference="link_southCameraBody">
     <material>Gazebo/Red</material>
   </gazebo>

File: cable_joint_description/urdf/cable_joint.urdf.xacro (robot description, xacro)
@@ -70,12 +70,12 @@
         </inertial>
     </link>
-    <joint name="joint_world_camerabody" type="revolute">
+    <joint name="joint_world_soucambody" type="revolute">
         <origin rpy="0 0 ${PI/2}" xyz="0 -0.5 ${L_CAMBODY/2}"/>
         <parent link="world"/>
-        <child link="link_cameraBody"/>
+        <child link="link_southCameraBody"/>
         <limit effort="0" lower="0" upper="0" velocity="0"/>
         <axis rpy="0 0 0" xyz="0 0 1"/>
     </joint>
-    <link name="link_cameraBody">
+    <link name="link_southCameraBody">
         <visual>
             <origin rpy="0 0 0" xyz="0 0 0"/>
@@ -97,12 +97,12 @@
         </inertial>
     </link>
-    <joint name="joint_camerabody_lens" type="revolute">
+    <joint name="joint_soucambody_soulens" type="revolute">
         <origin rpy="0 ${PI/2} 0" xyz="${L_CAMBODY/2+L_LENS/2} 0 0"/>
-        <parent link="link_cameraBody"/>
-        <child link="link_lens"/>
+        <parent link="link_southCameraBody"/>
+        <child link="link_southLens"/>
         <limit effort="0" lower="0" upper="0" velocity="0"/>
         <axis rpy="0 0 0" xyz="0 0 1"/>
     </joint>
-    <link name="link_lens">
+    <link name="link_southLens">
         <visual>
             <origin rpy="0 0 0" xyz="0 0 0"/>
@@ -124,11 +124,11 @@
         </inertial>
     </link>
-    <!-- camera needs to be rotated coreectly -->
-    <joint name="camera_optical_joint" type="fixed">
+    <!-- rotate optical link, x axis should be pointing to the view-->
+    <joint name="joint_soulens_souopt" type="fixed">
       <origin xyz="0 0 0" rpy="${-PI/2} ${-PI/2} ${PI/2}"/>
-      <parent link="link_lens"/>
-      <child link="link_optical"/>
-    </joint>
-    <link name="link_optical">
+      <parent link="link_southLens"/>
+      <child link="link_southOptical"/>
+    </joint>
+    <link name="link_southOptical">
     </link>
     <joint name="joint_base_eastpin" type="revolute">

Commit message: create west camera

File: cable_joint_description/urdf/cable_joint.gazebo.xacro (robot description, xacro)
@@ -1,9 +1,9 @@
 <?xml version="1.0"?>
 <robot>
-  <!-- camera -->
+  <!-- south camera -->
   <gazebo reference="link_southOptical">
     <sensor type="camera" name="camera1">
       <update_rate>30.0</update_rate>
-      <camera name="rgb">
+      <camera name="rgb_south">
         <horizontal_fov>1.3962634</horizontal_fov>
         <image>
@@ -28,8 +28,48 @@
         <alwaysOn>true</alwaysOn>
         <updateRate>0.0</updateRate>
-        <cameraName>cable_joint/rgb_camera</cameraName>
-        <imageTopicName>image_raw</imageTopicName>
-        <cameraInfoTopicName>camera_info</cameraInfoTopicName>
+        <cameraName>cable_joint/rgb_camera_south</cameraName>
+        <imageTopicName>south_image_raw</imageTopicName>
+        <cameraInfoTopicName>south_camera_info</cameraInfoTopicName>
         <frameName>link_southOptical</frameName>
+        <hackBaseline>0.07</hackBaseline>
+        <distortionK1>0.0</distortionK1>
+        <distortionK2>0.0</distortionK2>
+        <distortionK3>0.0</distortionK3>
+        <distortionT1>0.0</distortionT1>
+        <distortionT2>0.0</distortionT2>
+      </plugin>
+    </sensor>
+  </gazebo>
+  <!-- west camera -->
+  <gazebo reference="link_westOptical">
+    <sensor type="camera" name="camera2">
+      <update_rate>30.0</update_rate>
+      <camera name="rgb_west">
+        <horizontal_fov>1.3962634</horizontal_fov>
+        <image>
+          <width>800</width>
+          <height>800</height>
+          <format>R8G8B8</format>
+        </image>
+        <clip>
+          <near>0.02</near>
+          <far>300</far>
+        </clip>
+        <noise>
+          <type>gaussian</type>
+          <!-- Noise is sampled independently per pixel on each frame.
+               That pixel's noise value is added to each of its color
+               channels, which at that point lie in the range [0,1]. -->
+          <mean>0.0</mean>
+          <stddev>0.007</stddev>
+        </noise>
+      </camera>
+      <plugin name="camera_controller" filename="libgazebo_ros_camera.so">
+        <alwaysOn>true</alwaysOn>
+        <updateRate>0.0</updateRate>
+        <cameraName>cable_joint/rgb_camera_west</cameraName>
+        <imageTopicName>west_image_raw</imageTopicName>
+        <cameraInfoTopicName>west_camera_info</cameraInfoTopicName>
+        <frameName>link_westOptical</frameName>
         <hackBaseline>0.07</hackBaseline>
         <distortionK1>0.0</distortionK1>
@@ -63,4 +103,10 @@
   </gazebo>
   <gazebo reference="link_southCameraBody">
+    <material>Gazebo/Red</material>
+  </gazebo>
+  <gazebo reference="link_westLens">
+    <material>Gazebo/Black</material>
+  </gazebo>
+  <gazebo reference="link_westCameraBody">
     <material>Gazebo/Red</material>
   </gazebo>

File: cable_joint_description/urdf/cable_joint.urdf.xacro (robot description, xacro)
@@ -71,5 +71,5 @@
     </link>
     <joint name="joint_world_soucambody" type="revolute">
-        <origin rpy="0 0 ${PI/2}" xyz="0 -0.5 ${L_CAMBODY/2}"/>
+        <origin rpy="0 0 0" xyz="0 -0.5 ${L_CAMBODY}"/>
         <parent link="world"/>
         <child link="link_southCameraBody"/>
@@ -81,5 +81,5 @@
             <origin rpy="0 0 0" xyz="0 0 0"/>
             <geometry>
-                <box size="${L_CAMBODY} ${L_CAMBODY*2} ${L_CAMBODY*2}"/>
+                <box size="${L_CAMBODY*2} ${L_CAMBODY} ${L_CAMBODY*2}"/>
             </geometry>
             <material name="red"/>
@@ -88,5 +88,5 @@
             <origin rpy="0 0 0" xyz="0 0 0"/>
             <geometry>
-                <box size="${L_CAMBODY} ${L_CAMBODY*2} ${L_CAMBODY*2}"/>
+                <box size="${L_CAMBODY*2} ${L_CAMBODY} ${L_CAMBODY*2}"/>
             </geometry>
         </collision>
@@ -94,9 +94,9 @@
             <mass value="${M_CAMBODY}"/>
             <origin rpy="0 0 0" xyz="0 0 0"/>
-            <inertia ixx="${1/12*M_CAMBODY*(L_CAMBODY*L_CAMBODY*4+L_CAMBODY*L_CAMBODY*4)}" ixy="0" ixz="0" iyy="${1/12*M_CAMBODY*(L_CAMBODY*L_CAMBODY+L_CAMBODY*L_CAMBODY*4)}" iyz="0" izz="${1/12*M_CAMBODY*(L_CAMBODY*L_CAMBODY*4+L_CAMBODY*L_CAMBODY)}"/>
+            <inertia ixx="${1/12*M_CAMBODY*(L_CAMBODY*L_CAMBODY+L_CAMBODY*L_CAMBODY*4)}" ixy="0" ixz="0" iyy="${1/12*M_CAMBODY*(L_CAMBODY*L_CAMBODY*4+L_CAMBODY*L_CAMBODY*4)}" iyz="0" izz="${1/12*M_CAMBODY*(L_CAMBODY*L_CAMBODY*4+L_CAMBODY*L_CAMBODY)}"/>
         </inertial>
     </link>
     <joint name="joint_soucambody_soulens" type="revolute">
-        <origin rpy="0 ${PI/2} 0" xyz="${L_CAMBODY/2+L_LENS/2} 0 0"/>
+        <origin rpy="0 0 0" xyz="0 ${L_CAMBODY/2+L_LENS/2} 0"/>
         <parent link="link_southCameraBody"/>
         <child link="link_southLens"/>
@@ -106,5 +106,5 @@
     <link name="link_southLens">
         <visual>
-            <origin rpy="0 0 0" xyz="0 0 0"/>
+            <origin rpy="${PI/2} 0 0" xyz="0 0 0"/>
             <geometry>
                 <cylinder length="${L_LENS}" radius="${R_LENS}"/>
@@ -113,5 +113,5 @@
         </visual>
         <collision>
-            <origin rpy="0 0 0" xyz="0 0 0"/>
+            <origin rpy="${PI/2} 0 0" xyz="0 0 0"/>
             <geometry>
                 <cylinder length="${L_LENS}" radius="${R_LENS}"/>
@@ -120,5 +120,5 @@
         <inertial>
             <mass value="${M_LENS}"/>
-            <origin rpy="0 0 0" xyz="0 0 0"/>
+            <origin rpy="${PI/2} 0 0" xyz="0 0 0"/>
             <inertia ixx="${1/12*M_LENS*(3*R_LENS*R_LENS+L_LENS*L_LENS)}" ixy="0" ixz="0" iyy="${1/12*M_LENS*(3*R_LENS*R_LENS+L_LENS*L_LENS)}" iyz="0" izz="${1/2*M_LENS*R_LENS*R_LENS}"/>
         </inertial>
@@ -126,9 +126,71 @@
     <!-- rotate optical link, x axis should be pointing to the view-->
     <joint name="joint_soulens_souopt" type="fixed">
-      <origin xyz="0 0 0" rpy="${-PI/2} ${-PI/2} ${PI/2}"/>
+      <origin xyz="0 0 0" rpy="0 0 ${PI/2}"/>
       <parent link="link_southLens"/>
       <child link="link_southOptical"/>
     </joint>
     <link name="link_southOptical">
+    </link>
+    <joint name="joint_world_wescambody" type="revolute">
+        <origin rpy="0 0 0" xyz="-0.5 0 ${L_CAMBODY}"/>
+        <parent link="world"/>
+        <child link="link_westCameraBody"/>
+        <limit effort="0" lower="0" upper="0" velocity="0"/>
+        <axis rpy="0 0 0" xyz="0 0 1"/>
+    </joint>
+    <link name="link_westCameraBody">
+        <visual>
+            <origin rpy="0 0 0" xyz="0 0 0"/>
+            <geometry>
+                <box size="${L_CAMBODY} ${L_CAMBODY*2} ${L_CAMBODY*2}"/>
+            </geometry>
+            <material name="red"/>
+        </visual>
+        <collision>
+            <origin rpy="0 0 0" xyz="0 0 0"/>
+            <geometry>
+                <box size="${L_CAMBODY} ${L_CAMBODY*2} ${L_CAMBODY*2}"/>
+            </geometry>
+        </collision>
+        <inertial>
+            <mass value="${M_CAMBODY}"/>
+            <origin rpy="0 0 0" xyz="0 0 0"/>
+            <inertia ixx="${1/12*M_CAMBODY*(L_CAMBODY*L_CAMBODY*4+L_CAMBODY*L_CAMBODY*4)}" ixy="0" ixz="0" iyy="${1/12*M_CAMBODY*(L_CAMBODY*L_CAMBODY+L_CAMBODY*L_CAMBODY*4)}" iyz="0" izz="${1/12*M_CAMBODY*(L_CAMBODY*L_CAMBODY*4+L_CAMBODY*L_CAMBODY)}"/>
+        </inertial>
+    </link>
+    <joint name="joint_wescambody_weslens" type="revolute">
+        <origin rpy="0 0 0" xyz="${L_CAMBODY/2+L_LENS/2} 0 0"/>
+        <parent link="link_westCameraBody"/>
+        <child link="link_westLens"/>
+        <limit effort="0" lower="0" upper="0" velocity="0"/>
+        <axis rpy="0 0 0" xyz="0 0 1"/>
+    </joint>
+    <link name="link_westLens">
+        <visual>
+            <origin rpy="0 ${PI/2} 0" xyz="0 0 0"/>
+            <geometry>
+                <cylinder length="${L_LENS}" radius="${R_LENS}"/>
+            </geometry>
+            <material name="black"/>
+        </visual>
+        <collision>
+            <origin rpy="0 ${PI/2} 0" xyz="0 0 0"/>
+            <geometry>
+                <cylinder length="${L_LENS}" radius="${R_LENS}"/>
+            </geometry>
+        </collision>
+        <inertial>
+            <mass value="${M_LENS}"/>
+            <origin rpy="0 ${PI/2} 0" xyz="0 0 0"/>
+            <inertia ixx="${1/12*M_LENS*(3*R_LENS*R_LENS+L_LENS*L_LENS)}" ixy="0" ixz="0" iyy="${1/12*M_LENS*(3*R_LENS*R_LENS+L_LENS*L_LENS)}" iyz="0" izz="${1/2*M_LENS*R_LENS*R_LENS}"/>
+        </inertial>
+    </link>
+    <!-- rotate west optical link, x axis should be pointing to the view-->
+    <joint name="joint_weslens_wesopt" type="fixed">
+      <origin xyz="0 0 0" rpy="0 0 0"/>
+      <parent link="link_westLens"/>
+      <child link="link_westOptical"/>
+    </joint>
+    <link name="link_westOptical">
     </link>
     <joint name="joint_base_eastpin" type="revolute">
