Commit message: update link_base in urdf

File: cable_joint_description/urdf/cable_joint.urdf.xacro (robot description, xacro)
@@ -1,14 +1,22 @@
 <?xml version="1.0" ?>
 <robot name="cable_joint" xmlns:xacro="https://www.ros.org/wiki/xacro" >
-  <!-- Constants for robot dimensions -->
-  <xacro:property name="PI" value="3.1415926535897931"/>
-  <xacro:property name="body_length" value="0.02" /> <!-- Size of square 'camera' box -->
-  <!-- Import all Gazebo-customization elements, including Gazebo colors -->
-  <xacro:include filename="$(find cable_joint_description)/urdf/cable_joint.gazebo.xacro" />
-  <!-- Import Rviz colors -->
-  <xacro:include filename="$(find cable_joint_description)/urdf/materials.xacro" />
-  <!-- Used for fixing robot to Gazebo 'base_link' -->
-  <link name="world"/>
-  <joint name="joint_world_base" type="revolute">
+    <!-- Constants for robot dimensions -->
+    <xacro:property name="PI" value="3.1415926535897931"/>
+    <!-- properties of link_base -->
+    <xacro:property name="R_BASE" value="0.1"/>
+    <xacro:property name="L_BASE" value="0.02"/>
+    <xacro:property name="M_BASE" value="1000"/>
+    <!-- properties of link_base -->
+    <xacro:property name="R_BASE" value="0.1"/>
+    <xacro:property name="L_BASE" value="0.02"/>
+    <xacro:property name="M_BASE" value="1000"/>
+    <xacro:property name="body_length" value="0.02" /> <!-- Size of square 'camera' box -->
+    <!-- Import all Gazebo-customization elements, including Gazebo colors -->
+    <xacro:include filename="$(find cable_joint_description)/urdf/cable_joint.gazebo.xacro" />
+    <!-- Import Rviz colors -->
+    <xacro:include filename="$(find cable_joint_description)/urdf/materials.xacro" />
+    <!-- Used for fixing robot to Gazebo 'base_link' -->
+    <link name="world"/>
+    <!-- <joint name="joint_world_base" type="revolute">
     <origin rpy="0 0 0" xyz="0 0 0"/>
     <parent link="world"/>
@@ -16,26 +24,26 @@
     <limit effort="0" lower="0" upper="0" velocity="0"/>
     <axis rpy="0 0 0" xyz="0 0 1"/>
-  </joint>
-  <link name="link_base">
-    <collision>
-      <origin rpy="0 0 0" xyz="0 0 0"/>
-      <geometry>
-        <cylinder length="0.02" radius="0.1"/>
-      </geometry>
-    </collision>
-    <visual>
-      <origin rpy="0 0 0" xyz="0 0 0"/>
-      <geometry>
-        <cylinder length="0.02" radius="0.1"/>
-      </geometry>
-      <material name="black"/>
-    </visual>
-    <inertial>
-      <mass value="1000"/>
-      <origin rpy="0 0 0" xyz="0 0 0"/>
-      <inertia ixx="2.533" ixy="0" ixz="0" iyy="2.533" iyz="0" izz="5.236"/>
-    </inertial>
-  </link>
-  <joint name="joint_world_camerabody" type="revolute">
+    </joint> -->
+    <link name="link_base">
+        <visual>
+            <origin rpy="0 0 0" xyz="0 0 0"/>
+            <geometry>
+                <cylinder length="{L_BASE}" radius="${R_BASE}"/>
+            </geometry>
+        <material name="black"/>
+        </visual>
+        <collision>
+            <origin rpy="0 0 0" xyz="0 0 0"/>
+            <geometry>
+                <cylinder length="${L_BASE}" radius="${R_BASE}"/>
+            </geometry>
+        </collision>
+        <inertial>
+            <mass value="1000"/>
+            <origin rpy="0 0 0" xyz="0 0 0"/>
+            <inertia ixx="${1/12*M_BASE*(3*R_HAT*R_HAT+L_HAT*L_HAT)}" ixy="0" ixz="0" iyy="${1/12*M_BASE*(3*R_HAT*R_HAT+L_HAT*L_HAT)}" iyz="0" izz="${1/2*M_BASE*R_HAT*R_HAT}"/>
+        </inertial>
+    </link>
+    <joint name="joint_world_camerabody" type="revolute">
     <origin rpy="0 0 ${PI/2}" xyz="0 -0.5 ${body_length/2}"/>
     <parent link="world"/>
@@ -43,5 +51,5 @@
     <limit effort="0" lower="0" upper="0" velocity="0"/>
     <axis rpy="0 0 0" xyz="0 0 1"/>
-  </joint>
+    </joint>
   <link name="link_camera_body">
     <collision>

Commit message: create camera body link in cable joint model

File: cable_joint_description/urdf/cable_joint.urdf.xacro (robot description, xacro)
@@ -11,5 +11,7 @@
     <xacro:property name="L_BASE" value="0.02"/>
     <xacro:property name="M_BASE" value="1000"/>
-    <xacro:property name="body_length" value="0.02" /> <!-- Size of square 'camera' box -->
+    <!-- properties of link_camera_body -->
+    <xacro:property name="L_CAMBODY" value="0.02"/>
+    <xacro:property name="M_CAMBODY" value="0.1"/>
     <!-- Import all Gazebo-customization elements, including Gazebo colors -->
     <xacro:include filename="$(find cable_joint_description)/urdf/cable_joint.gazebo.xacro" />
@@ -18,16 +20,13 @@
     <!-- Used for fixing robot to Gazebo 'base_link' -->
     <link name="world"/>
-    <!-- <joint name="joint_world_base" type="revolute">
-    <origin rpy="0 0 0" xyz="0 0 0"/>
-    <parent link="world"/>
-    <child link="link_base"/>
-    <limit effort="0" lower="0" upper="0" velocity="0"/>
-    <axis rpy="0 0 0" xyz="0 0 1"/>
-    </joint> -->
+    <joint name="joint_world_base" type="fixed">
+        <parent link="world"/>
+        <child link="link_base"/>
+    </joint>
     <link name="link_base">
         <visual>
             <origin rpy="0 0 0" xyz="0 0 0"/>
             <geometry>
-                <cylinder length="{L_BASE}" radius="${R_BASE}"/>
+                <cylinder length="${L_BASE}" radius="${R_BASE}"/>
             </geometry>
         <material name="black"/>
@@ -42,393 +41,33 @@
             <mass value="1000"/>
             <origin rpy="0 0 0" xyz="0 0 0"/>
-            <inertia ixx="${1/12*M_BASE*(3*R_HAT*R_HAT+L_HAT*L_HAT)}" ixy="0" ixz="0" iyy="${1/12*M_BASE*(3*R_HAT*R_HAT+L_HAT*L_HAT)}" iyz="0" izz="${1/2*M_BASE*R_HAT*R_HAT}"/>
+            <inertia ixx="${1/12*M_BASE*(3*R_BASE*R_BASE+L_BASE*L_BASE)}" ixy="0" ixz="0" iyy="${1/12*M_BASE*(3*R_BASE*R_BASE+L_BASE*L_BASE)}" iyz="0" izz="${1/2*M_BASE*R_BASE*R_BASE}"/>
         </inertial>
     </link>
     <joint name="joint_world_camerabody" type="revolute">
-    <origin rpy="0 0 ${PI/2}" xyz="0 -0.5 ${body_length/2}"/>
-    <parent link="world"/>
-    <child link="link_camera_body"/>
-    <limit effort="0" lower="0" upper="0" velocity="0"/>
-    <axis rpy="0 0 0" xyz="0 0 1"/>
+        <origin rpy="0 0 ${PI/2}" xyz="0 -0.5 ${L_CAMBODY/2}"/>
+        <parent link="world"/>
+        <child link="link_camera_body"/>
+        <limit effort="0" lower="0" upper="0" velocity="0"/>
+        <axis rpy="0 0 0" xyz="0 0 1"/>
     </joint>
-  <!-- <link name="link_camera_body">
-    <collision>
-      <origin rpy="0 0 0" xyz="0 -0.5 0"/>
-      <geometry>
-        <box size="${body_length} ${body_length*2} ${body_length*2}"/>
-      </geometry>
-    </collision>
-    <visual>
-      <origin rpy="0 0 0" xyz="0 0 0"/>
-      <geometry>
-        <box size="${body_length} ${body_length*2} ${body_length*2}"/>
-      </geometry>
-      <material name="red"/>
-    </visual>
-    <inertial>
-      <mass value="0.1"/>
-      <origin rpy="0 0 0" xyz="0 0 0"/>
-      <inertia ixx="1e-6" ixy="0" ixz="0" iyy="1e-6" iyz="0" izz="1e-6"/>
-    </inertial>
-  </link>
-  <joint name="joint_camerabody_lens" type="revolute">
-    <origin rpy="0 ${PI/2} 0" xyz="${body_length/2+body_length/16} 0 0"/>
-    <parent link="link_camera_body"/>
-    <child link="link_lens"/>
-    <limit effort="0" lower="0" upper="0" velocity="0"/>
-    <axis rpy="0 0 0" xyz="0 0 1"/>
-  </joint>
-  <link name="link_lens">
-    <collision>
-      <origin rpy="0 0 0" xyz="0 -0.5 0"/>
-      <geometry>
-        <cylinder length="${body_length/8}" radius="${body_length/2}"/>
-      </geometry>
-    </collision>
-    <visual>
-      <origin rpy="0 0 0" xyz="0 0 0"/>
-      <geometry>
-        <cylinder length="${body_length/8}" radius="${body_length/2}"/>
-      </geometry>
-      <material name="black"/>
-    </visual>
-    <inertial>
-      <mass value="0.01"/>
-      <origin rpy="0 0 0" xyz="0 0 0"/>
-      <inertia ixx="1e-6" ixy="0" ixz="0" iyy="1e-6" iyz="0" izz="1e-6"/>
-    </inertial>
-  </link>
-  <!-- camera needs to be rotated coreectly -->
-  <joint name="camera_optical_joint" type="fixed">
-    <origin xyz="0 0 0" rpy="${-PI/2} ${-PI/2} ${PI/2}"/>
-    <parent link="link_lens"/>
-    <child link="link_optical"/>
-  </joint>
-  <link name="link_optical">
-  </link>
-  <joint name="joint_base_lowersupport" type="revolute">
-    <origin rpy="0 0 0" xyz="0 0 0"/>
-    <limit effort="0" lower="0" upper="0" velocity="0"/>
-    <axis rpy="0 0 0" xyz="0 0 1"/>
-    <parent link="link_base"/>
-    <child link="link_lower_support"/>
-    <origin rpy="0 0 0" xyz="0 0 0.01"/>
-  </joint>
-  <link name="link_lower_support">
-    <collision>
-      <origin rpy="0 0 0" xyz="0 0 0.07"/>
-      <geometry>
-        <cylinder length="0.14" radius="0.015"/>
-      </geometry>
-    </collision>
-    <visual>
-      <origin rpy="0 0 0" xyz="0 0 0.07"/>
-      <geometry>
-        <cylinder length="0.14" radius="0.015"/>
-      </geometry>
-      <material name="grey"/>
-    </visual>
-    <inertial>
-      <mass value="100"/>
-      <origin rpy="0 0 0" xyz="0 0 0"/>
-      <inertia ixx="0.1" ixy="0" ixz="0" iyy="0.1" iyz="0" izz="0.1"/>
-    </inertial>
-  </link>
-  <joint name="joint_base_pinwest" type="revolute">
-    <parent link="link_base"/>
-    <child link="link_pin_west"/>
-    <origin rpy="0 0 0" xyz="-0.1 0 0.01"/>
-    <limit effort="0" lower="0" upper="0" velocity="0"/>
-    <axis rpy="0 0 0" xyz="0 0 1"/>
-  </joint>
-  <link name="link_pin_west">
-    <collision>
-      <origin rpy="0 0 0" xyz="0 0 0"/>
-      <geometry>
-        <sphere radius="0.02"/>
-      </geometry>
-    </collision>
-    <visual>
-      <origin rpy="0 0 0" xyz="0 0 0"/>
-      <geometry>
-        <sphere radius="0.02"/>
-      </geometry>
-      <material name="red"/>
-    </visual>
-    <inertial>
-      <mass value="1"/>
-      <origin rpy="0 0 0" xyz="0 0 0"/>
-      <inertia ixx="1e-4" ixy="0" ixz="0" iyy="1e-4" iyz="0" izz="1e-4"/>
-    </inertial>
-  </link>
-  <joint name="joint_base_pineast" type="revolute">
-    <parent link="link_base"/>
-    <child link="link_pin_east"/>
-    <origin rpy="0 0 0" xyz="0.1 0 0.01"/>
-    <limit effort="0" lower="0" upper="0" velocity="0"/>
-    <axis rpy="0 0 0" xyz="0 0 1"/>
-  </joint>
-  <link name="link_pin_east">
-    <collision>
-      <origin rpy="0 0 0" xyz="0 0 0"/>
-      <geometry>
-        <sphere radius="0.02"/>
-      </geometry>
-    </collision>
-    <visual>
-      <origin rpy="0 0 0" xyz="0 0 0"/>
-      <geometry>
-        <sphere radius="0.02"/>
-      </geometry>
-      <material name="blue"/>
-    </visual>
-    <inertial>
-      <mass value="1"/>
-      <origin rpy="0 0 0" xyz="0 0 0"/>
-      <inertia ixx="1e-4" ixy="0" ixz="0" iyy="1e-4" iyz="0" izz="1e-4"/>
-    </inertial>
-  </link>
-  <joint name="joint_lowersupport_ballroll" type="revolute">
-    <parent link="link_lower_support"/>
-    <child link="link_ball_roll"/>
-    <origin rpy="0 0 0" xyz="0 0 0.14"/>
-    <axis xyz="1 0 0"/>
-    <limit effort="10" velocity="${PI*2}" lower="${-4*PI/9}" upper="${4*PI/9}"/>
-  </joint>
-  <link name="link_ball_roll">
-    <collision>
-      <origin rpy="0 0 0" xyz="0 0 0"/>
-      <geometry>
-        <sphere radius="0.00001"/>
-      </geometry>
-    </collision>
-    <visual>
-      <origin rpy="0 0 0" xyz="0 0 0"/>
-      <geometry>
-        <sphere radius="0.00001"/>
-      </geometry>
-      <material name="white"/>
-    </visual>
-    <inertial>
-      <mass value="0.1"/>
-      <origin rpy="0 0 0" xyz="0 0 0"/>
-      <inertia ixx="1e-8" ixy="0" ixz="0" iyy="1e-8" iyz="0" izz="1e-8"/>
-    </inertial>
-  </link>
-  <joint name="joint_ballroll_ballpitch" type="revolute">
-    <parent link="link_ball_roll"/>
-    <child link="link_ball_pitch"/>
-    <origin rpy="0 0 0" xyz="0 0 0"/>
-    <axis xyz="0 1 0"/>
-    <limit effort="10" velocity="${PI*2}" lower="${-4*PI/9}" upper="${4*PI/9}"/>
-  </joint>
-  <link name="link_ball_pitch">
-    <collision>
-      <origin rpy="0 0 0" xyz="0 0 0"/>
-      <geometry>
-        <sphere radius="0.00001"/>
-      </geometry>
-    </collision>
-    <visual>
-      <origin rpy="0 0 0" xyz="0 0 0"/>
-      <geometry>
-        <sphere radius="0.00001"/>
-      </geometry>
-      <material name="white"/>
-    </visual>
-    <inertial>
-      <mass value="0.1"/>
-      <origin rpy="0 0 0" xyz="0 0 0"/>
-      <inertia ixx="1e-8" ixy="0" ixz="0" iyy="1e-8" iyz="0" izz="1e-8"/>
-    </inertial>
-  </link>
-  <joint name="joint_ballpitch_ballyaw" type="revolute">
-    <parent link="link_ball_pitch"/>
-    <child link="link_ball_yaw"/>
-    <origin rpy="0 0 0" xyz="0 0 0"/>
-    <axis xyz="0 0 1"/>
-    <limit effort="10" velocity="${PI*2}" lower="${-PI/8}" upper="${PI/8}"/>
-  </joint>
-  <link name="link_ball_yaw">
-    <collision>
-      <origin rpy="0 0 0" xyz="0 0 0"/>
-      <geometry>
-        <sphere radius="0.02"/>
-      </geometry>
-    </collision>
-    <visual>
-      <origin rpy="0 0 0" xyz="0 0 0"/>
-      <geometry>
-        <sphere radius="0.02"/>
-      </geometry>
-      <material name="yellow"/>
-    </visual>
-    <inertial>
-      <mass value="1"/>
-      <origin rpy="0 0 0" xyz="0 0 0"/>
-      <inertia ixx="1e-6" ixy="0" ixz="0" iyy="1e-6" iyz="0" izz="1e-6"/>
-    </inertial>
-  </link>
-  <joint name="joint_ballyaw_uppersupport" type="revolute">
-    <origin rpy="0 0 0" xyz="0 0 0.03"/>
-    <limit effort="0" lower="0" upper="0" velocity="0"/>
-    <axis xyz="0 0 1"/>
-    <parent link="link_ball_yaw"/>
-    <child link="link_upper_support"/>
-  </joint>
-  <link name="link_upper_support">
-    <collision>
-      <origin rpy="0 0 0" xyz="0 0 0"/>
-      <geometry>
-        <cylinder length="0.04" radius="0.01"/>
-      </geometry>
-    </collision>
-    <visual>
-      <origin rpy="0 0 0" xyz="0 0 0"/>
-      <geometry>
-        <cylinder length="0.04" radius="0.01"/>
-      </geometry>
-      <material name="grey"/>
-    </visual>
-    <inertial>
-      <mass value="1e-5"/>
-      <origin rpy="0 0 0" xyz="0 0 0"/>
-      <inertia ixx="1e-8" ixy="0" ixz="0" iyy="1e-8" iyz="0" izz="1e-8"/>
-    </inertial>
-  </link>
-  <joint name="joint_uppersupport_disc" type="revolute">
-    <origin rpy="0 0 0" xyz="0 0 0.02"/>
-    <limit effort="0" lower="0" upper="0" velocity="0"/>
-    <axis xyz="0 0 1"/>
-    <parent link="link_upper_support"/>
-    <child link="link_disc"/>
-  </joint>
-  <link name="link_disc">
-    <collision>
-      <origin rpy="0 0 0" xyz="0 0 0"/>
-      <geometry>
-        <cylinder length="0.02" radius="0.1"/>
-      </geometry>
-    </collision>
-    <visual>
-      <origin rpy="0 0 0" xyz="0 0 0"/>
-      <geometry>
-        <cylinder length="0.02" radius="0.1"/>
-      </geometry>
-      <material name="white"/>
-    </visual>
-    <inertial>
-      <mass value="0.0001"/>
-      <origin rpy="0 0 0" xyz="0 0 0"/>
-      <inertia ixx="1e-6" ixy="0" ixz="0" iyy="1e-6" iyz="0" izz="1e-6"/>
-    </inertial>
-  </link>
-  <joint name="joint_disc_cubenortheast" type="revolute">
-    <parent link="link_disc"/>
-    <child link="link_cube_northeast"/>
-    <origin rpy="0 0 0" xyz="0.0707 0.0707 0"/>
-    <limit effort="0" lower="0" upper="0" velocity="0"/>
-    <axis rpy="0 0 0" xyz="0 0 1"/>
-  </joint>
-  <link name="link_cube_northeast">
-    <collision>
-      <origin rpy="0 0 0" xyz="0 0 0"/>
-      <geometry>
-        <box size="0.02 0.02 0.02" />
-      </geometry>
-    </collision>
-    <visual>
-      <origin rpy="0 0 0" xyz="0 0 0"/>
-      <geometry>
-        <box size="0.02 0.02 0.02" />
-      </geometry>
-      <material name="purple"/>
-    </visual>
-    <inertial>
-      <mass value="1e-5"/>
-      <origin rpy="0 0 0" xyz="0 0 0"/>
-      <inertia ixx="1e-8" ixy="0" ixz="0" iyy="1e-8" iyz="0" izz="1e-8"/>
-    </inertial>
-  </link>
-  <joint name="joint_disc_cubenorthwest" type="revolute">
-    <parent link="link_disc"/>
-    <child link="link_cube_northwest"/>
-    <origin rpy="0 0 0" xyz="-0.0707 0.0707 0"/>
-    <limit effort="0" lower="0" upper="0" velocity="0"/>
-    <axis rpy="0 0 0" xyz="0 0 1"/>
-  </joint>
-  <link name="link_cube_northwest">
-    <collision>
-      <origin rpy="0 0 0" xyz="0 0 0"/>
-      <geometry>
-        <box size="0.02 0.02 0.02" />
-      </geometry>
-    </collision>
-    <visual>
-      <origin rpy="0 0 0" xyz="0 0 0"/>
-      <geometry>
-        <box size="0.02 0.02 0.02" />
-      </geometry>
-      <material name="red"/>
-    </visual>
-    <inertial>
-      <mass value="1e-5"/>
-      <origin rpy="0 0 0" xyz="0 0 0"/>
-      <inertia ixx="1e-8" ixy="0" ixz="0" iyy="1e-8" iyz="0" izz="1e-8"/>
-    </inertial>
-  </link>
-  <joint name="joint_disc_cubesouthwest" type="revolute">
-    <parent link="link_disc"/>
-    <child link="link_cube_southwest"/>
-    <origin rpy="0 0 0" xyz="-0.0707 -0.0707 0"/>
-    <limit effort="0" lower="0" upper="0" velocity="0"/>
-    <axis rpy="0 0 0" xyz="0 0 1"/>
-  </joint>
-  <link name="link_cube_southwest">
-    <collision>
-      <origin rpy="0 0 0" xyz="0 0 0"/>
-      <geometry>
-        <box size="0.02 0.02 0.02" />
-      </geometry>
-    </collision>
-    <visual>
-      <origin rpy="0 0 0" xyz="0 0 0"/>
-      <geometry>
-        <box size="0.02 0.02 0.02" />
-      </geometry>
-      <material name="orange"/>
-    </visual>
-    <inertial>
-      <mass value="1e-5"/>
-      <origin rpy="0 0 0" xyz="0 0 0"/>
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
Commit message: continue update cable joint urdf

File: cable_joint_description/urdf/cable_joint.urdf.xacro (robot description, xacro)
@@ -14,4 +14,15 @@
     <xacro:property name="L_CAMBODY" value="0.02"/>
     <xacro:property name="M_CAMBODY" value="0.1"/>
+    <!-- properties of link_lens_body -->
+    <xacro:property name="R_LENS" value="0.02"/>
+    <xacro:property name="L_LENS" value="0.002"/>
+    <xacro:property name="M_LENS" value="0.01"/>
+    <!-- properties of link_pin's -->
+    <xacro:property name="R_PIN" value="0.02"/>
+    <xacro:property name="M_PIN" value="1"/>
+    <!-- properties of link_lowerSupport -->
+    <xacro:property name="R_LOWSUPPORT" value="0.015"/>
+    <xacro:property name="L_LOWSUPPORT" value="0.14"/>
+    <xacro:property name="M_LOWSUPPORT" value="10"/>
     <!-- Import all Gazebo-customization elements, including Gazebo colors -->
     <xacro:include filename="$(find cable_joint_description)/urdf/cable_joint.gazebo.xacro" />
@@ -71,3 +82,120 @@
         </inertial>
     </link>
+    <joint name="joint_camerabody_lens" type="revolute">
+        <origin rpy="0 ${PI/2} 0" xyz="${L_CAMBODY/2+L_LENS/2} 0 0"/>
+        <parent link="link_camera_body"/>
+        <child link="link_lens"/>
+        <limit effort="0" lower="0" upper="0" velocity="0"/>
+        <axis rpy="0 0 0" xyz="0 0 1"/>
+    </joint>
+    <link name="link_lens">
+        <visual>
+            <origin rpy="0 0 0" xyz="0 0 0"/>
+            <geometry>
+                <cylinder length="${L_LENS}" radius="${R_LENS}"/>
+            </geometry>
+            <material name="black"/>
+        </visual>
+        <collision>
+            <origin rpy="0 0 0" xyz="0 0 0"/>
+            <geometry>
+                <cylinder length="${L_LENS}" radius="${R_LENS}"/>
+            </geometry>
+        </collision>
+        <inertial>
+            <mass value="${M_LENS}"/>
+            <origin rpy="0 0 0" xyz="0 0 0"/>
+            <inertia ixx="${1/12*M_LENS*(3*R_LENS*R_LENS+L_LENS*L_LENS)}" ixy="0" ixz="0" iyy="${1/12*M_LENS*(3*R_LENS*R_LENS+L_LENS*L_LENS)}" iyz="0" izz="${1/2*M_LENS*R_LENS*R_LENS}"/>
+        </inertial>
+    </link>
+    <!-- camera needs to be rotated coreectly -->
+    <joint name="camera_optical_joint" type="fixed">
+      <origin xyz="0 0 0" rpy="${-PI/2} ${-PI/2} ${PI/2}"/>
+      <parent link="link_lens"/>
+      <child link="link_optical"/>
+    </joint>
+    <link name="link_optical">
+    </link>
+    <joint name="joint_base_eastpin" type="revolute">
+        <parent link="link_base"/>
+        <child link="link_eastPin"/>
+        <origin rpy="0 0 0" xyz="${R_BASE} 0 ${L_BASE/2}"/>
+        <limit effort="0" lower="0" upper="0" velocity="0"/>
+        <axis rpy="0 0 0" xyz="0 0 1"/>
+    </joint>
+    <link name="link_eastPin">
+        <visual>
+            <origin rpy="0 0 0" xyz="0 0 0"/>
+            <geometry>
+                <sphere radius="${R_PIN}"/>
+            </geometry>
+            <material name="blue"/>
+        </visual>
+        <collision>
+            <origin rpy="0 0 0" xyz="0 0 0"/>
+            <geometry>
+                <sphere radius="${R_PIN}"/>
+            </geometry>
+        </collision>
+        <inertial>
+            <mass value="${M_PIN}"/>
+            <origin rpy="0 0 0" xyz="0 0 0"/>
+            <inertia ixx="${2/5*M_PIN*R_PIN*R_PIN}" ixy="0" ixz="0" iyy="${2/5*M_PIN*R_PIN*R_PIN}" iyz="0" izz="${2/5*M_PIN*R_PIN*R_PIN}"/>
+        </inertial>
+    </link>
+    <joint name="joint_base_westpin" type="revolute">
+        <parent link="link_base"/>
+        <child link="link_westPin"/>
+        <origin rpy="0 0 0" xyz="${-R_BASE} 0 ${L_BASE/2}"/>
+        <limit effort="0" lower="0" upper="0" velocity="0"/>
+        <axis rpy="0 0 0" xyz="0 0 1"/>
+    </joint>
+    <link name="link_westPin">
+        <visual>
+            <origin rpy="0 0 0" xyz="0 0 0"/>
+            <geometry>
+                <sphere radius="${R_PIN}"/>
+            </geometry>
+            <material name="red"/>
+        </visual>
+        <collision>
+            <origin rpy="0 0 0" xyz="0 0 0"/>
+            <geometry>
+                <sphere radius="${R_PIN}"/>
+            </geometry>
+        </collision>
+        <inertial>
+            <mass value="${M_PIN}"/>
+            <origin rpy="0 0 0" xyz="0 0 0"/>
+            <inertia ixx="${2/5*M_PIN*R_PIN*R_PIN}" ixy="0" ixz="0" iyy="${2/5*M_PIN*R_PIN*R_PIN}" iyz="0" izz="${2/5*M_PIN*R_PIN*R_PIN}"/>
+        </inertial>
+    </link>
+    <joint name="joint_base_lowersupport" type="revolute">
+        <origin rpy="0 0 0" xyz="0 0 0"/>
+        <limit effort="0" lower="0" upper="0" velocity="0"/>
+        <axis rpy="0 0 0" xyz="0 0 1"/>
+        <parent link="link_base"/>
+        <child link="link_lowerSupport"/>
+        <origin rpy="0 0 0" xyz="0 0 0.01"/>
+    </joint>
+    <link name="link_lowerSupport">
+        <visual>
+            <origin rpy="0 0 0" xyz="0 0 0.07"/>
+            <geometry>
+                <cylinder length="${L_LOWSUPPORT}" radius="${R_LOWSUPPORT}"/>
+            </geometry>
+            <material name="grey"/>
+        </visual>
+        <collision>
+            <origin rpy="0 0 0" xyz="0 0 0.07"/>
+            <geometry>
+                <cylinder length="${L_LOWSUPPORT}" radius="${R_LOWSUPPORT}"/>
+            </geometry>
+        </collision>
+        <inertial>
+            <mass value="${M_LOWSUPPORT}"/>
+            <origin rpy="0 0 0" xyz="0 0 0"/>
+            <inertia ixx="${1/12*M_LOWSUPPORT*(3*R_LOWSUPPORT*R_LOWSUPPORT+L_LOWSUPPORT*L_LOWSUPPORT)}" ixy="0" ixz="0" iyy="${1/12*M_LOWSUPPORT*(3*R_LOWSUPPORT*R_LOWSUPPORT+L_LOWSUPPORT*L_LOWSUPPORT)}" iyz="0" izz="${1/2*M_LOWSUPPORT*R_LOWSUPPORT*R_LOWSUPPORT}"/>
+        </inertial>
+    </link>
 </robot>
