Commit message: create first hidden rod for ball joint

File: cable_joint_description/urdf/cable_joint.urdf.xacro (robot description, xacro)
@@ -6,9 +6,5 @@
     <xacro:property name="R_BASE" value="0.1"/>
     <xacro:property name="L_BASE" value="0.02"/>
-    <xacro:property name="M_BASE" value="1000"/>
-    <!-- properties of link_base -->
-    <xacro:property name="R_BASE" value="0.1"/>
-    <xacro:property name="L_BASE" value="0.02"/>
-    <xacro:property name="M_BASE" value="1000"/>
+    <xacro:property name="M_BASE" value="10"/>
     <!-- properties of link_camera_body -->
     <xacro:property name="L_CAMBODY" value="0.02"/>
@@ -24,5 +20,9 @@
     <xacro:property name="R_LOWSUPPORT" value="0.015"/>
     <xacro:property name="L_LOWSUPPORT" value="0.14"/>
-    <xacro:property name="M_LOWSUPPORT" value="10"/>
+    <xacro:property name="M_LOWSUPPORT" value="1"/>
+    <!-- properties of link_hiddenRod -->
+    <xacro:property name="R_LOWSUPPORT" value="0.000001"/>
+    <xacro:property name="L_LOWSUPPORT" value="0.000004"/>
+    <xacro:property name="M_LOWSUPPORT" value="0.00001"/>
     <!-- Import all Gazebo-customization elements, including Gazebo colors -->
     <xacro:include filename="$(find cable_joint_description)/urdf/cable_joint.gazebo.xacro" />
@@ -199,3 +199,30 @@
         </inertial>
     </link>
+    <joint name="joint_lowersupport_hiddenballroll" type="revolute">
+        <parent link="link_lower_support"/>
+        <child link="link_hiddenBallRoll"/>
+        <origin rpy="0 0 0" xyz="0 0 0.14"/>
+        <axis xyz="1 0 0"/>
+        <limit effort="10" velocity="${PI*2}" lower="${-4*PI/9}" upper="${4*PI/9}"/>
+    </joint>
+    <link name="link_hiddenBallRoll">
+        <visual>
+            <origin rpy="0 0 0" xyz="0 0 0"/>
+            <geometry>
+                <sphere radius="0.00001"/>
+            </geometry>
+            <material name="white"/>
+        </visual>
+        <collision>
+            <origin rpy="0 0 0" xyz="0 0 0"/>
+            <geometry>
+                <sphere radius="0.00001"/>
+            </geometry>
+        </collision>
+                <inertial>
+            <mass value="0.1"/>
+            <origin rpy="0 0 0" xyz="0 0 0"/>
+            <inertia ixx="1e-8" ixy="0" ixz="0" iyy="1e-8" iyz="0" izz="1e-8"/>
+        </inertial>
+    </link>
 </robot>

Commit message: create ball joint

File: cable_joint_description/urdf/cable_joint.urdf.xacro (robot description, xacro)
@@ -3,4 +3,5 @@
     <!-- Constants for robot dimensions -->
     <xacro:property name="PI" value="3.1415926535897931"/>
+    <xacro:property name="EPSILON" value="1e-8"/>
     <!-- properties of link_base -->
     <xacro:property name="R_BASE" value="0.1"/>
@@ -21,8 +22,11 @@
     <xacro:property name="L_LOWSUPPORT" value="0.14"/>
     <xacro:property name="M_LOWSUPPORT" value="1"/>
-    <!-- properties of link_hiddenRod -->
-    <xacro:property name="R_LOWSUPPORT" value="0.000001"/>
-    <xacro:property name="L_LOWSUPPORT" value="0.000004"/>
-    <xacro:property name="M_LOWSUPPORT" value="0.00001"/>
+    <!-- properties of link_hiddenLink -->
+    <xacro:property name="R_HIDLINK" value="0.000001"/>
+    <xacro:property name="L_HIDLINK" value="0.000004"/>
+    <xacro:property name="M_HIDLINK" value="0.00001"/>
+    <!-- properties of link_ball -->
+    <xacro:property name="R_BALL" value="0.04"/>
+    <xacro:property name="M_BALL" value="1"/>
     <!-- Import all Gazebo-customization elements, including Gazebo colors -->
     <xacro:include filename="$(find cable_joint_description)/urdf/cable_joint.gazebo.xacro" />
@@ -199,29 +203,83 @@
         </inertial>
     </link>
-    <joint name="joint_lowersupport_hiddenballroll" type="revolute">
-        <parent link="link_lower_support"/>
-        <child link="link_hiddenBallRoll"/>
-        <origin rpy="0 0 0" xyz="0 0 0.14"/>
+    <joint name="joint_lowersupport_hiddenlinkroll" type="revolute">
+        <parent link="link_lowerSupport"/>
+        <child link="link_hiddenLinkRoll"/>
+        <origin rpy="0 0 0" xyz="0 0 ${L_LOWSUPPORT}"/>
         <axis xyz="1 0 0"/>
-        <limit effort="10" velocity="${PI*2}" lower="${-4*PI/9}" upper="${4*PI/9}"/>
-    </joint>
-    <link name="link_hiddenBallRoll">
-        <visual>
-            <origin rpy="0 0 0" xyz="0 0 0"/>
-            <geometry>
-                <sphere radius="0.00001"/>
+        <limit effort="10" velocity="${PI*2}" lower="${-PI+EPSILON}" upper="${PI-EPSILON}"/>
+    </joint>
+    <link name="link_hiddenLinkRoll">
+        <visual>
+            <origin rpy="${PI/2} 0 0" xyz="0 0 0"/>
+            <geometry>
+                <cylinder length="${L_HIDLINK}" radius="${R_HIDLINK}"/>
             </geometry>
             <material name="white"/>
         </visual>
         <collision>
-            <origin rpy="0 0 0" xyz="0 0 0"/>
-            <geometry>
-                <sphere radius="0.00001"/>
-            </geometry>
-        </collision>
-                <inertial>
-            <mass value="0.1"/>
-            <origin rpy="0 0 0" xyz="0 0 0"/>
-            <inertia ixx="1e-8" ixy="0" ixz="0" iyy="1e-8" iyz="0" izz="1e-8"/>
+            <origin rpy="${PI/2} 0 0" xyz="0 0 0"/>
+            <geometry>
+                <cylinder length="${L_HIDLINK}" radius="${R_HIDLINK}"/>
+            </geometry>
+        </collision>
+        <inertial>
+            <mass value="${M_HIDLINK}"/>
+            <origin rpy="${PI/2} 0 0" xyz="0 0 0"/>
+            <inertia ixx="${1/12*M_HIDLINK*(3*R_HIDLINK*R_HIDLINK+L_HIDLINK*L_HIDLINK)}" ixy="0" ixz="0" iyy="${1/12*M_HIDLINK*(3*R_HIDLINK*R_HIDLINK+L_HIDLINK*L_HIDLINK)}" iyz="0" izz="${1/2*M_HIDLINK*R_HIDLINK*R_HIDLINK}"/>
+        </inertial>
+    </link>
+    <joint name="joint_hiddenlinkroll_hiddenlinkpitch" type="revolute">
+        <parent link="link_hiddenLinkRoll"/>
+        <child link="link_hiddenLinkPitch"/>
+        <origin rpy="0 0 0" xyz="0 0 ${R_HIDLINK}"/>
+        <axis xyz="0 1 0"/>
+        <limit effort="10" velocity="${PI*2}" lower="${-PI+EPSILON}" upper="${PI-EPSILON}"/>
+    </joint>
+    <link name="link_hiddenLinkPitch">
+        <visual>
+            <origin rpy="0 ${PI/2} 0" xyz="0 0 0"/>
+            <geometry>
+                <cylinder length="${L_HIDLINK}" radius="${R_HIDLINK}"/>
+            </geometry>
+            <material name="white"/>
+        </visual>
+        <collision>
+            <origin rpy="0 ${PI/2} 0" xyz="0 0 0"/>
+            <geometry>
+                <cylinder length="${L_HIDLINK}" radius="${R_HIDLINK}"/>
+            </geometry>
+        </collision>
+        <inertial>
+            <mass value="${M_HIDLINK}"/>
+            <origin rpy="0 ${PI/2} 0" xyz="0 0 0"/>
+            <inertia ixx="${1/12*M_HIDLINK*(3*R_HIDLINK*R_HIDLINK+L_HIDLINK*L_HIDLINK)}" ixy="0" ixz="0" iyy="${1/12*M_HIDLINK*(3*R_HIDLINK*R_HIDLINK+L_HIDLINK*L_HIDLINK)}" iyz="0" izz="${1/2*M_HIDLINK*R_HIDLINK*R_HIDLINK}"/>
+        </inertial>
+    </link>
+    <joint name="joint_hiddenlinkpitch_ball" type="revolute">
+        <parent link="link_hiddenLinkPitch"/>
+        <child link="link_ball"/>
+        <origin rpy="0 0 0" xyz="0 0 ${R_HIDLINK}"/>
+        <axis xyz="0 0 1"/>
+        <limit effort="10" velocity="${PI*2}" lower="${-PI+EPSILON}" upper="${PI-EPSILON}"/>
+    </joint>
+    <link name="link_ball">
+        <visual>
+            <origin rpy="0 0 ${PI/2}" xyz="0 0 0"/>
+            <geometry>
+                <sphere radius="${R_BALL}"/>
+            </geometry>
+            <material name="white"/>
+        </visual>
+        <collision>
+            <origin rpy="0 0 ${PI/2}" xyz="0 0 0"/>
+            <geometry>
+                <sphere radius="${R_BALL}"/>
+            </geometry>
+        </collision>
+        <inertial>
+            <mass value="${M_BALL}"/>
+            <origin rpy="0 0 ${PI/2}" xyz="0 0 0"/>
+            <inertia ixx="${2/5*M_BALL*R_BALL*R_BALL}" ixy="0" ixz="0" iyy="${2/5*M_BALL*R_BALL*R_BALL}" iyz="0" izz="${2/5*M_BALL*R_BALL*R_BALL}"/>
         </inertial>
     </link>

Commit message: create upper support link

File: cable_joint_description/urdf/cable_joint.urdf.xacro (robot description, xacro)
@@ -29,4 +29,8 @@
     <xacro:property name="R_BALL" value="0.04"/>
     <xacro:property name="M_BALL" value="1"/>
+    <!-- properties of link_lowerSupport -->
+    <xacro:property name="R_UPPSUPPORT" value="0.01"/>
+    <xacro:property name="L_UPPSUPPORT" value="0.08"/>
+    <xacro:property name="M_UPPSUPPORT" value="0.1"/>
     <!-- Import all Gazebo-customization elements, including Gazebo colors -->
     <xacro:include filename="$(find cable_joint_description)/urdf/cable_joint.gazebo.xacro" />
@@ -284,3 +288,30 @@
         </inertial>
     </link>
+    <joint name="joint_ball_uppersupport" type="revolute">
+          <origin rpy="0 0 0" xyz="0 0 ${R_BALL}"/>
+          <limit effort="0" lower="0" upper="0" velocity="0"/>
+          <axis xyz="0 0 1"/>
+          <parent link="link_ball"/>
+          <child link="link_upperSupport"/>
+    </joint>
+    <link name="link_upperSupport">
+        <visual>
+            <origin rpy="0 0 0" xyz="0 0 0"/>
+            <geometry>
+                <cylinder length="${L_UPPSUPPORT}" radius="${R_UPPSUPPORT}"/>
+            </geometry>
+            <material name="grey"/>
+        </visual>
+    <collision>
+        <origin rpy="0 0 0" xyz="0 0 0"/>
+        <geometry>
+            <cylinder length="${L_UPPSUPPORT}" radius="${R_UPPSUPPORT}"/>
+        </geometry>
+    </collision>
+    <inertial>
+        <mass value="1e-5"/>
+        <origin rpy="0 0 0" xyz="0 0 0"/>
+        <inertia ixx="${1/12*M_UPPSUPPORT*(3*R_UPPSUPPORT*R_UPPSUPPORT+L_UPPSUPPORT*L_UPPSUPPORT)}" ixy="0" ixz="0" iyy="${1/12*M_UPPSUPPORT*(3*R_UPPSUPPORT*R_UPPSUPPORT+L_UPPSUPPORT*L_UPPSUPPORT)}" iyz="0" izz="${1/2*M_UPPSUPPORT*R_UPPSUPPORT*R_UPPSUPPORT}"/>
+      </inertial>
+    </link>
 </robot>

Commit message: finish cable joint v2 urdf

File: cable_joint_description/urdf/cable_joint.urdf.xacro (robot description, xacro)
@@ -29,8 +29,15 @@
     <xacro:property name="R_BALL" value="0.04"/>
     <xacro:property name="M_BALL" value="1"/>
-    <!-- properties of link_lowerSupport -->
+    <!-- properties of link_upperSupport -->
     <xacro:property name="R_UPPSUPPORT" value="0.01"/>
     <xacro:property name="L_UPPSUPPORT" value="0.08"/>
     <xacro:property name="M_UPPSUPPORT" value="0.1"/>
+    <!-- properties of link_disc -->
+    <xacro:property name="R_DISC" value="0.1"/>
+    <xacro:property name="L_DISC" value="0.02"/>
+    <xacro:property name="M_DISC" value="0.1"/>
+    <!-- properties of link_camera_body -->
+    <xacro:property name="L_CUBE" value="0.02"/>
+    <xacro:property name="M_CUBE" value="0.001"/>
     <!-- Import all Gazebo-customization elements, including Gazebo colors -->
     <xacro:include filename="$(find cable_joint_description)/urdf/cable_joint.gazebo.xacro" />
@@ -310,8 +317,143 @@
     </collision>
     <inertial>
-        <mass value="1e-5"/>
+        <mass value="${M_UPPSUPPORT}"/>
         <origin rpy="0 0 0" xyz="0 0 0"/>
         <inertia ixx="${1/12*M_UPPSUPPORT*(3*R_UPPSUPPORT*R_UPPSUPPORT+L_UPPSUPPORT*L_UPPSUPPORT)}" ixy="0" ixz="0" iyy="${1/12*M_UPPSUPPORT*(3*R_UPPSUPPORT*R_UPPSUPPORT+L_UPPSUPPORT*L_UPPSUPPORT)}" iyz="0" izz="${1/2*M_UPPSUPPORT*R_UPPSUPPORT*R_UPPSUPPORT}"/>
       </inertial>
     </link>
+    <joint name="joint_uppersupport_disc" type="revolute">
+          <origin rpy="0 0 0" xyz="0 0 ${L_UPPSUPPORT/2}"/>
+          <limit effort="0" lower="0" upper="0" velocity="0"/>
+          <axis xyz="0 0 1"/>
+          <parent link="link_upperSupport"/>
+          <child link="link_disc"/>
+    </joint>
+    <link name="link_disc">
+        <visual>
+            <origin rpy="0 0 0" xyz="0 0 0"/>
+            <geometry>
+                <cylinder length="${L_DISC}" radius="${R_DISC}"/>
+              </geometry>
+              <material name="white"/>
+        </visual>
+        <collision>
+            <origin rpy="0 0 0" xyz="0 0 0"/>
+            <geometry>
+                <cylinder length="${L_DISC}" radius="${R_DISC}"/>
+            </geometry>
+        </collision>
+        <inertial>
+            <mass value="${M_DISC}"/>
+            <origin rpy="0 0 0" xyz="0 0 0"/>
+            <inertia ixx="${1/12*M_DISC*(3*R_DISC*R_DISC+L_DISC*L_DISC)}" ixy="0" ixz="0" iyy="${1/12*M_DISC*(3*R_DISC*R_DISC+L_DISC*L_DISC)}" iyz="0" izz="${1/2*M_DISC*R_DISC*R_DISC}"/>
+        </inertial>
+    </link>
+    <joint name="joint_disc_necube" type="revolute">
+          <parent link="link_disc"/>
+          <child link="link_northeastCube"/>
+          <origin rpy="0 0 0" xyz="0.0707 0.0707 0"/>
+          <limit effort="0" lower="0" upper="0" velocity="0"/>
+          <axis rpy="0 0 0" xyz="0 0 1"/>
+    </joint>
+    <link name="link_northeastCube">
+        <visual>
+            <origin rpy="0 0 0" xyz="0 0 0"/>
+            <geometry>
+                <box size="${L_CUBE} ${L_CUBE} ${L_CUBE}" />
+            </geometry>
+            <material name="purple"/>
+        </visual>
+        <collision>
+            <origin rpy="0 0 0" xyz="0 0 0"/>
+            <geometry>
+                <box size="${L_CUBE} ${L_CUBE} ${L_CUBE}"/>
+            </geometry>
+        </collision>
+        <inertial>
+            <mass value="${M_CUBE}"/>
+            <origin rpy="0 0 0" xyz="0 0 0"/>
+            <inertia ixx="${1/12*M_CUBE*(L_CUBE*L_CUBE+L_CUBE*L_CUBE)}" ixy="0" ixz="0" iyy="${1/12*M_CUBE*(L_CUBE*L_CUBE+L_CUBE*L_CUBE)}" iyz="0" izz="${1/12*M_CUBE*(L_CUBE*L_CUBE+L_CUBE*L_CUBE)}"/>
+      </inertial>
+    </link>
+    <joint name="joint_disc_nwcube" type="revolute">
+          <parent link="link_disc"/>
+          <child link="link_northwestCube"/>
+          <origin rpy="0 0 0" xyz="-0.0707 0.0707 0"/>
+          <limit effort="0" lower="0" upper="0" velocity="0"/>
+          <axis rpy="0 0 0" xyz="0 0 1"/>
+    </joint>
+    <link name="link_northwestCube">
+        <visual>
+            <origin rpy="0 0 0" xyz="0 0 0"/>
+            <geometry>
+                <box size="${L_CUBE} ${L_CUBE} ${L_CUBE}" />
+            </geometry>
+            <material name="seance"/>
+        </visual>
+        <collision>
+            <origin rpy="0 0 0" xyz="0 0 0"/>
+            <geometry>
+                <box size="${L_CUBE} ${L_CUBE} ${L_CUBE}"/>
+            </geometry>
+        </collision>
+        <inertial>
+            <mass value="${M_CUBE}"/>
+            <origin rpy="0 0 0" xyz="0 0 0"/>
+            <inertia ixx="${1/12*M_CUBE*(L_CUBE*L_CUBE+L_CUBE*L_CUBE)}" ixy="0" ixz="0" iyy="${1/12*M_CUBE*(L_CUBE*L_CUBE+L_CUBE*L_CUBE)}" iyz="0" izz="${1/12*M_CUBE*(L_CUBE*L_CUBE+L_CUBE*L_CUBE)}"/>
+      </inertial>
+    </link>
+    <joint name="joint_disc_swcube" type="revolute">
+          <parent link="link_disc"/>
+          <child link="link_southwestCube"/>
+          <origin rpy="0 0 0" xyz="-0.0707 -0.0707 0"/>
+          <limit effort="0" lower="0" upper="0" velocity="0"/>
+          <axis rpy="0 0 0" xyz="0 0 1"/>
+    </joint>
+    <link name="link_southwestCube">
+        <visual>
+            <origin rpy="0 0 0" xyz="0 0 0"/>
+            <geometry>
+                <box size="${L_CUBE} ${L_CUBE} ${L_CUBE}" />
+            </geometry>
+            <material name="orange"/>
+        </visual>
+        <collision>
+            <origin rpy="0 0 0" xyz="0 0 0"/>
+            <geometry>
+                <box size="${L_CUBE} ${L_CUBE} ${L_CUBE}"/>
+            </geometry>
+        </collision>
+        <inertial>
+            <mass value="${M_CUBE}"/>
+            <origin rpy="0 0 0" xyz="0 0 0"/>
+            <inertia ixx="${1/12*M_CUBE*(L_CUBE*L_CUBE+L_CUBE*L_CUBE)}" ixy="0" ixz="0" iyy="${1/12*M_CUBE*(L_CUBE*L_CUBE+L_CUBE*L_CUBE)}" iyz="0" izz="${1/12*M_CUBE*(L_CUBE*L_CUBE+L_CUBE*L_CUBE)}"/>
+      </inertial>
+    </link>
+    <joint name="joint_disc_secube" type="revolute">
+          <parent link="link_disc"/>
+          <child link="link_southeastCube"/>
+          <origin rpy="0 0 0" xyz="0.0707 -0.0707 0"/>
+          <limit effort="0" lower="0" upper="0" velocity="0"/>
+          <axis rpy="0 0 0" xyz="0 0 1"/>
+    </joint>
+    <link name="link_southeastCube">
+        <visual>
+            <origin rpy="0 0 0" xyz="0 0 0"/>
+            <geometry>
+                <box size="${L_CUBE} ${L_CUBE} ${L_CUBE}" />
+            </geometry>
+            <material name="sky"/>
+        </visual>
+        <collision>
+            <origin rpy="0 0 0" xyz="0 0 0"/>
+            <geometry>
+                <box size="${L_CUBE} ${L_CUBE} ${L_CUBE}"/>
+            </geometry>
+        </collision>
+        <inertial>
+            <mass value="${M_CUBE}"/>
+            <origin rpy="0 0 0" xyz="0 0 0"/>
+            <inertia ixx="${1/12*M_CUBE*(L_CUBE*L_CUBE+L_CUBE*L_CUBE)}" ixy="0" ixz="0" iyy="${1/12*M_CUBE*(L_CUBE*L_CUBE+L_CUBE*L_CUBE)}" iyz="0" izz="${1/12*M_CUBE*(L_CUBE*L_CUBE+L_CUBE*L_CUBE)}"/>
+      </inertial>
+    </link>
 </robot>

Commit message: add camera north

File: cable_joint_description/urdf/cable_joint.urdf.xacro (robot description, xacro)
@@ -41,5 +41,5 @@
     <xacro:property name="M_CUBE" value="0.001"/>
     <!-- Import all Gazebo-customization elements, including Gazebo colors -->
-    <xacro:include filename="$(find cable_joint_description)/urdf/cable_joint.gazebo.xacro" />
+    <xacro:include filename="$(find cable_joint_description)/urdf/cable_joint.gazebo" />
     <!-- Import Rviz colors -->
     <xacro:include filename="$(find cable_joint_description)/urdf/materials.xacro" />
@@ -193,4 +193,66 @@
     </joint>
     <link name="link_westOptical">
+    </link>
+    <joint name="joint_world_norcambody" type="revolute">
+        <origin rpy="0 0 0" xyz="0 0.5 ${L_CAMBODY}"/>
+        <parent link="world"/>
+        <child link="link_northCameraBody"/>
+        <limit effort="0" lower="0" upper="0" velocity="0"/>
+        <axis rpy="0 0 0" xyz="0 0 1"/>
+    </joint>
+    <link name="link_northCameraBody">
+        <visual>
+            <origin rpy="0 0 0" xyz="0 0 0"/>
+            <geometry>
+                <box size="${L_CAMBODY*2} ${L_CAMBODY} ${L_CAMBODY*2}"/>
+            </geometry>
+            <material name="red"/>
+        </visual>
+        <collision>
+            <origin rpy="0 0 0" xyz="0 0 0"/>
+            <geometry>
+                <box size="${L_CAMBODY*2} ${L_CAMBODY} ${L_CAMBODY*2}"/>
+            </geometry>
+        </collision>
+        <inertial>
+            <mass value="${M_CAMBODY}"/>
+            <origin rpy="0 0 0" xyz="0 0 0"/>
+            <inertia ixx="${1/12*M_CAMBODY*(L_CAMBODY*L_CAMBODY+L_CAMBODY*L_CAMBODY*4)}" ixy="0" ixz="0" iyy="${1/12*M_CAMBODY*(L_CAMBODY*L_CAMBODY*4+L_CAMBODY*L_CAMBODY*4)}" iyz="0" izz="${1/12*M_CAMBODY*(L_CAMBODY*L_CAMBODY*4+L_CAMBODY*L_CAMBODY)}"/>
+        </inertial>
+    </link>
+    <joint name="joint_norcambody_norlens" type="revolute">
+        <origin rpy="0 0 0" xyz="0 -${L_CAMBODY/2+L_LENS/2} 0"/>
+        <parent link="link_northCameraBody"/>
+        <child link="link_northLens"/>
+        <limit effort="0" lower="0" upper="0" velocity="0"/>
+        <axis rpy="0 0 0" xyz="0 0 1"/>
+    </joint>
+    <link name="link_northLens">
+        <visual>
+            <origin rpy="${PI/2} 0 0" xyz="0 0 0"/>
+            <geometry>
+                <cylinder length="${L_LENS}" radius="${R_LENS}"/>
+            </geometry>
+            <material name="black"/>
+        </visual>
+        <collision>
+            <origin rpy="${PI/2} 0 0" xyz="0 0 0"/>
+            <geometry>
+                <cylinder length="${L_LENS}" radius="${R_LENS}"/>
+            </geometry>
+        </collision>
+        <inertial>
+            <mass value="${M_LENS}"/>
+            <origin rpy="${PI/2} 0 0" xyz="0 0 0"/>
+            <inertia ixx="${1/12*M_LENS*(3*R_LENS*R_LENS+L_LENS*L_LENS)}" ixy="0" ixz="0" iyy="${1/12*M_LENS*(3*R_LENS*R_LENS+L_LENS*L_LENS)}" iyz="0" izz="${1/2*M_LENS*R_LENS*R_LENS}"/>
+        </inertial>
+    </link>
+    <!-- rotate optical link, x axis should be pointing to the view-->
+    <joint name="joint_norlens_noropt" type="fixed">
+      <origin xyz="0 0 0" rpy="0 0 -${PI/2}"/>
+      <parent link="link_northLens"/>
+      <child link="link_northOptical"/>
+    </joint>
+    <link name="link_northOptical">
     </link>
     <joint name="joint_base_eastpin" type="revolute">
