Commit message: add east camera

File: cable_joint_description/urdf/cable_joint.urdf.xacro (robot description, xacro)
@@ -71,5 +71,5 @@
     </link>
     <joint name="joint_world_soucambody" type="revolute">
-        <origin rpy="0 0 0" xyz="0 -0.5 ${L_CAMBODY}"/>
+        <origin rpy="0 0 0" xyz="0 -0.5 ${L_CAMBODY/2}"/>
         <parent link="world"/>
         <child link="link_southCameraBody"/>
@@ -133,5 +133,5 @@
     </link>
     <joint name="joint_world_wescambody" type="revolute">
-        <origin rpy="0 0 0" xyz="-0.5 0 ${L_CAMBODY}"/>
+        <origin rpy="0 0 0" xyz="-0.5 0 ${L_CAMBODY/2}"/>
         <parent link="world"/>
         <child link="link_westCameraBody"/>
@@ -195,5 +195,5 @@
     </link>
     <joint name="joint_world_norcambody" type="revolute">
-        <origin rpy="0 0 0" xyz="0 0.5 ${L_CAMBODY}"/>
+        <origin rpy="0 0 0" xyz="0 0.5 ${L_CAMBODY/2}"/>
         <parent link="world"/>
         <child link="link_northCameraBody"/>
@@ -255,4 +255,66 @@
     </joint>
     <link name="link_northOptical">
+    </link>
+    <joint name="joint_world_eascambody" type="revolute">
+        <origin rpy="0 0 0" xyz="0.5 0 ${L_CAMBODY/2}"/>
+        <parent link="world"/>
+        <child link="link_eastCameraBody"/>
+        <limit effort="0" lower="0" upper="0" velocity="0"/>
+        <axis rpy="0 0 0" xyz="0 0 1"/>
+    </joint>
+    <link name="link_eastCameraBody">
+        <visual>
+            <origin rpy="0 0 0" xyz="0 0 0"/>
+            <geometry>
+                <box size="${L_CAMBODY} ${L_CAMBODY*2} ${L_CAMBODY*2}"/>
+            </geometry>
+            <material name="red"/>
+        </visual>
+        <collision>
+            <origin rpy="0 0 0" xyz="0 0 0"/>
+            <geometry>
+                <box size="${L_CAMBODY} ${L_CAMBODY*2} ${L_CAMBODY*2}"/>
+            </geometry>
+        </collision>
+        <inertial>
+            <mass value="${M_CAMBODY}"/>
+            <origin rpy="0 0 0" xyz="0 0 0"/>
+            <inertia ixx="${1/12*M_CAMBODY*(L_CAMBODY*L_CAMBODY*4+L_CAMBODY*L_CAMBODY*4)}" ixy="0" ixz="0" iyy="${1/12*M_CAMBODY*(L_CAMBODY*L_CAMBODY+L_CAMBODY*L_CAMBODY*4)}" iyz="0" izz="${1/12*M_CAMBODY*(L_CAMBODY*L_CAMBODY*4+L_CAMBODY*L_CAMBODY)}"/>
+        </inertial>
+    </link>
+    <joint name="joint_eascambody_easlens" type="revolute">
+        <origin rpy="0 0 0" xyz="-${L_CAMBODY/2+L_LENS/2} 0 0"/>
+        <parent link="link_eastCameraBody"/>
+        <child link="link_eastLens"/>
+        <limit effort="0" lower="0" upper="0" velocity="0"/>
+        <axis rpy="0 0 0" xyz="0 0 1"/>
+    </joint>
+    <link name="link_eastLens">
+        <visual>
+            <origin rpy="0 ${PI/2} 0" xyz="0 0 0"/>
+            <geometry>
+                <cylinder length="${L_LENS}" radius="${R_LENS}"/>
+            </geometry>
+            <material name="black"/>
+        </visual>
+        <collision>
+            <origin rpy="0 ${PI/2} 0" xyz="0 0 0"/>
+            <geometry>
+                <cylinder length="${L_LENS}" radius="${R_LENS}"/>
+            </geometry>
+        </collision>
+        <inertial>
+            <mass value="${M_LENS}"/>
+            <origin rpy="0 ${PI/2} 0" xyz="0 0 0"/>
+            <inertia ixx="${1/12*M_LENS*(3*R_LENS*R_LENS+L_LENS*L_LENS)}" ixy="0" ixz="0" iyy="${1/12*M_LENS*(3*R_LENS*R_LENS+L_LENS*L_LENS)}" iyz="0" izz="${1/2*M_LENS*R_LENS*R_LENS}"/>
+        </inertial>
+    </link>
+    <!-- rotate east optical link, x axis should be pointing to the view-->
+    <joint name="joint_easlens_easopt" type="fixed">
+      <origin xyz="0 0 0" rpy="0 0 ${PI}"/>
+      <parent link="link_eastLens"/>
+      <child link="link_eastOptical"/>
+    </joint>
+    <link name="link_eastOptical">
     </link>
     <joint name="joint_base_eastpin" type="revolute">
